Commit message: Added gazebo plugins

File: roomba_description/urdf/roomba.urdf (robot description, URDF)
Before this commit: robot create, 3 links, 2 joints
Joints:
- removed joint create__left_wheel
- removed joint create__right_wheel
- added joint create_left_wheel_hinge: type revolute, parent create__base, child create__left_wheel, origin xyz=0     0.13   0.032 rpy=0  0  0, axis 0  1  0, limit lower=0 upper=100 effort=100 velocity=10
- added joint create_right_wheel_hinge: type revolute, parent create__base, child create__right_wheel, origin xyz=0    -0.13   0.032 rpy=0  0  0, axis 0  1  0, limit lower=0 upper=100 effort=100 velocity=10
